File: 19-0002-01_Rev_B/DesignData.kicad_pcb (KiCad board)
At the start: 2 copper layers, 178 x 202 mm, 320 parts, among them J1 Conn_01x04_Male, SW11 SW_Push_45deg, SW12 SW_Push_45deg, SW13 SW_Push_45deg, SW14 SW_Push_45deg, SW15 SW_Push_45deg, SW16 SW_Push_45deg, SW17 SW_Push_45deg, SW21 SW_Push_45deg, SW22 SW_Push_45deg, SW23 SW_Push_45deg, SW24 SW_Push_45deg, SW25 SW_Push_45deg, SW26 SW_Push_45deg, SW27 SW_Push_45deg, SW32 SW_Push_45deg, SW33 SW_Push_45deg, SW34 SW_Push_45deg, SW35 SW_Push_45deg, SW36 SW_Push_45deg, U1 ESP32-Modul_AZ, U100 HT16K33_Modul, U101 SC56-11, U102 SC56-11, U103 SC56-11, U104 SC56-11, U105 SC56-11, U106 HT16K33_Modul, U2 ESP32-Modul_NodeMCU, U200 HT16K33_Modul, U201 SC56-11, U202 SC56-11, U203 SC56-11, U204 SC56-11, U205 SC56-11, U300 HT16K33_Modul, U301 SC56-11, U302 SC56-11, U303 SC56-11, U304 SC56-11, U305 SC56-11, U400 HT16K33_Modul, U401 SC56-11, U402 SC56-11, U403 SC56-11, U404 SC56-11, U405 SC56-11, U406 SC56-11

Commit message: in work
Other:
- board text added: "+5V"
- board text added: "GND"
Changed lines of the file:
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@@
   (general
     (thickness 1.6)
-    (drawings 329)
+    (drawings 331)
     (tracks 2891)
     (zones 0)
@@
     )
   )
+  (gr_text GND (at 149.698 155.037) (layer F.SilkS)
+    (effects (font (size 1.5 1.5) (thickness 0.3)))
+  )
+  (gr_text +5V (at 149.317 141.956) (layer F.SilkS)
+    (effects (font (size 1.5 1.5) (thickness 0.3)))
+  )
   (gr_text RSET (at 281.27 198.09) (layer F.SilkS)
     (effects (font (size 1.5 1.5) (thickness 0.3)))
@@
   (segment (start 247.996 102.586) (end 247.996 106.606728) (width 0.2) (layer F.Cu) (net 7))
   (segment (start 246.726 101.316) (end 247.996 102.586) (width 0.2) (layer F.Cu) (net 7))
-  (segment (start 259.807005 107.031005) (end 259.807 107.031) (width 0.2) (layer B.Cu) (net 23))
-  (segment (start 242.02599 107.031) (end 242.025998 107.030992) (width 0.2) (layer B.Cu) (net 20))
   (segment (start 284.826 101.316) (end 284.826 106.523004) (width 0.2) (layer F.Cu) (net 7))
-  (segment (start 259.382736 107.031) (end 259.807 107.031) (width 0.2) (layer B.Cu) (net 23))
-  (segment (start 256.506006 107.030992) (end 256.506014 107.031) (width 0.2) (layer B.Cu) (net 21))
   (segment (start 216.5 115.435998) (end 214.976 113.911998) (width 0.2) (layer F.Cu) (net 7))
   (segment (start 214.976 113.911998) (end 214.976 108.936) (width 0.2) (layer F.Cu) (net 7))
@@
   (segment (start 241.646 134.59) (end 241.646 131.288) (width 0.2) (layer F.Cu) (net 18))
   (segment (start 241.646 131.288) (end 241.646 128.748) (width 0.2) (layer F.Cu) (net 18))
+  (segment (start 242.02599 107.031) (end 242.025998 107.030992) (width 0.2) (layer B.Cu) (net 20))
   (segment (start 219.04 106.396) (end 219.04 107.52737) (width 0.2) (layer F.Cu) (net 20))
   (segment (start 218.64737 108.936) (end 219.04 108.936) (width 0.2) (layer F.Cu) (net 20))
@@
   (segment (start 240.249 108.809) (end 240.846001 108.211999) (width 0.2) (layer B.Cu) (net 20))
   (segment (start 221.664001 107.835999) (end 224.162999 107.835999) (width 0.2) (layer B.Cu) (net 20))
+  (segment (start 256.506006 107.030992) (end 256.506014 107.031) (width 0.2) (layer B.Cu) (net 21))
   (segment (start 235.380001 120.704001) (end 235.079999 120.403999) (width 0.2) (layer B.Cu) (net 21))
   (segment (start 238.259999 120.704001) (end 235.380001 120.704001) (width 0.2) (layer B.Cu) (net 21))
@@
   (segment (start 256.886 109.952) (end 256.886 112.237992) (width 0.2) (layer F.Cu) (net 21))
   (segment (start 256.886 109.952) (end 256.886 107.412) (width 0.2) (layer F.Cu) (net 21))
+  (segment (start 259.807005 107.031005) (end 259.807 107.031) (width 0.2) (layer B.Cu) (net 23))
+  (segment (start 259.382736 107.031) (end 259.807 107.031) (width 0.2) (layer B.Cu) (net 23))
   (segment (start 258.579999 118.503999) (end 258.880001 118.804001) (width 0.2) (layer B.Cu) (net 23))
   (segment (start 255.700001 118.503999) (end 258.579999 118.503999) (width 0.2) (layer B.Cu) (net 23))
@@
   (segment (start 235.72027 90.393994) (end 235.296006 90.393994) (width 0.2) (layer B.Cu) (net 43))
   (segment (start 235.720276 90.394) (end 235.72027 90.393994) (width 0.2) (layer B.Cu) (net 43))
+  (segment (start 256.586001 85.741003) (end 256.886 85.441004) (width 0.2) (layer F.Cu) (net 43))
+  (segment (start 256.885996 85.441) (end 256.886 85.441004) (width 0.2) (layer B.Cu) (net 43))
+  (segment (start 256.886 90.394) (end 256.886 86.076) (width 0.2) (layer F.Cu) (net 43))
   (segment (start 219.04 85.06) (end 219.04 86.19137) (width 0.2) (layer F.Cu) (net 44))
   (segment (start 220.564 87.6) (end 219.04 87.6) (width 0.2) (layer F.Cu) (net 44))
@@
   (segment (start 251.806 44.05063) (end 251.806 42.896) (width 0.2) (layer F.Cu) (net 47))
   (segment (start 251.806 45.182) (end 251.806 44.05063) (width 0.2) (layer F.Cu) (net 47))
+  (via (at 268.315992 42.896) (size 0.6) (drill 0.3) (layers F.Cu B.Cu) (net 47))
+  (segment (start 268.315992 36.292008) (end 268.315992 42.471736) (width 0.2) (layer F.Cu) (net 47))
+  (segment (start 268.315992 42.471736) (end 268.315992 42.896) (width 0.2) (layer F.Cu) (net 47))
+  (segment (start 269.586 50.262) (end 268.315992 48.991992) (width 0.2) (layer F.Cu) (net 47))
+  (segment (start 268.315992 48.991992) (end 268.315992 43.320264) (width 0.2) (layer F.Cu) (net 47))
+  (segment (start 269.586 35.022) (end 268.315992 36.292008) (width 0.2) (layer F.Cu) (net 47))
+  (segment (start 252.230264 42.896) (end 268.315992 42.896) (width 0.2) (layer B.Cu) (net 47))
+  (segment (start 268.315992 43.320264) (end 268.315992 42.896) (width 0.2) (layer F.Cu) (net 47))
+  (segment (start 251.806 42.896) (end 252.230264 42.896) (width 0.2) (layer B.Cu) (net 47))
   (segment (start 268.786001 52.510001) (end 269.586 53.31) (width 0.2) (layer B.Cu) (net 48))
   (segment (start 268.485999 52.209999) (end 268.786001 52.510001) (width 0.2) (layer B.Cu) (net 48))
@@
   (via (at 282.286 87.6) (size 0.6) (drill 0.3) (layers F.Cu B.Cu) (net 52))
   (segment (start 254.346 87.6) (end 282.286 87.6) (width 0.2) (layer B.Cu) (net 52))
+  (segment (start 254.346 87.6) (end 254.346 86.076) (width 0.2) (layer F.Cu) (net 52))
   (via (at 251.806 88.616) (size 0.6) (drill 0.3) (layers F.Cu B.Cu) (net 53))
   (segment (start 251.806 88.616) (end 251.806 86.203) (width 0.2) (layer F.Cu) (net 53))
-  (segment (start 256.586001 85.741003) (end 256.886 85.441004) (width 0.2) (layer F.Cu) (net 43))
-  (segment (start 256.885996 85.441) (end 256.886 85.441004) (width 0.2) (layer B.Cu) (net 43))
-  (segment (start 256.886 90.394) (end 256.886 86.076) (width 0.2) (layer F.Cu) (net 43))
-  (via (at 268.315992 42.896) (size 0.6) (drill 0.3) (layers F.Cu B.Cu) (net 47))
-  (segment (start 268.315992 36.292008) (end 268.315992 42.471736) (width 0.2) (layer F.Cu) (net 47))
-  (segment (start 268.315992 42.471736) (end 268.315992 42.896) (width 0.2) (layer F.Cu) (net 47))
-  (segment (start 269.586 50.262) (end 268.315992 48.991992) (width 0.2) (layer F.Cu) (net 47))
-  (segment (start 268.315992 48.991992) (end 268.315992 43.320264) (width 0.2) (layer F.Cu) (net 47))
-  (segment (start 269.586 35.022) (end 268.315992 36.292008) (width 0.2) (layer F.Cu) (net 47))
-  (segment (start 252.230264 42.896) (end 268.315992 42.896) (width 0.2) (layer B.Cu) (net 47))
-  (segment (start 268.315992 43.320264) (end 268.315992 42.896) (width 0.2) (layer F.Cu) (net 47))
-  (segment (start 251.806 42.896) (end 252.230264 42.896) (width 0.2) (layer B.Cu) (net 47))
-  (segment (start 254.346 87.6) (end 254.346 86.076) (width 0.2) (layer F.Cu) (net 52))
   (via (at 270.856002 88.616) (size 0.6) (drill 0.3) (layers F.Cu B.Cu) (net 53))
   (segment (start 251.806 88.616) (end 270.856002 88.616) (width 0.2) (layer B.Cu) (net 53))
